File: AtMEGA328p/Schematic/fan controller.kicad_pcb (KiCad board)
At the start: 2 copper layers, 31.8 x 43.2 mm, 7 parts, among them J1 Conn_02x05_Counter_Clockwise, M1 Fan, Q1 2N7000, U1 ATmega328P-PU

Commit message: updated schematic
Parts:
- removed M1: Fan, Connector_PinHeader_2.54mm:PinHeader_1x02_P2.54mm_Vertical
- added C2: 0.1u, Capacitor_THT:C_Disc_D10.0mm_W2.5mm_P5.00mm, F.Cu at (143.5, 80.0)
- added Fan: Fan, Connector_PinHeader_2.54mm:PinHeader_1x02_P2.54mm_Vertical, F.Cu at (147.3, 83.8)
- added Power: PinHeader_1x02_P2.54mm_Vertical, Connector_PinHeader_2.54mm:PinHeader_1x02_P2.54mm_Vertical, F.Cu at (147.3, 76.2)
- added UART: PinHeader_1x02_P2.54mm_Vertical, Connector_PinHeader_2.54mm:PinHeader_1x02_P2.54mm_Vertical, F.Cu at (147.3, 67.3)
- moved Q1 2.54 mm to (138.4, 82.5)
- moved C1 1.27 mm to (123.2, 85.1)
- renumbered C2 to C1, J1 to Prog
Connections:
- Prog pad 1: Net-(J1-Pad1) -> Net-(J1-Pad5)
- Prog pad 2: Net-(J1-Pad2) -> Net-(C2-Pad1)
- Prog pad 3: Net-(J1-Pad3) -> Net-(J1-Pad4)
- Prog pad 4: Net-(J1-Pad4) -> Net-(C2-Pad1)
- Prog pad 5: Net-(J1-Pad5) -> Net-(J1-Pad3)
- Prog pad 6: Net-(C2-Pad2) -> Net-(C2-Pad1)
- Prog pad 7: Net-(C2-Pad2) -> Net-(C2-Pad1)
- Prog pad 8: Net-(C2-Pad2) -> Net-(C2-Pad1)
- Prog pad 9: Net-(C2-Pad2) -> Net-(J1-Pad1)
- Q1 pad 1: Net-(C2-Pad2) -> Net-(C2-Pad1)
Routing:
- net Net-(C2-Pad2): track 20.4 -> 62.8 mm
- net Net-(U1-Pad3): track 0.00 -> 22.3 mm
- net Net-(U1-Pad2): track 0.00 -> 22.3 mm
- net Net-(J1-Pad3): track 33.0 -> 38.3 mm
- net Net-(J1-Pad4): track 10.4 -> 6.66 mm
- net Net-(M1-Pad2): track 6.35 -> 9.42 mm
- net Net-(J1-Pad1): track 6.66 -> 8.45 mm
- net Net-(J1-Pad5): track 6.66 -> 5.61 mm
- net Net-(Q1-Pad2): track 18.7 -> 17.7 mm
- net (no net): vias 0 -> 17
- added copper zone on B.Cu, net Net-(C2-Pad1)
