File: AtMEGA328p/Schematic/fan controller.sch (KiCad schematic (older format))
At the start: 8 parts, among them J1 Conn_02x05_Counter_Clockwise, M1 Fan, Q1 2N7000, U1 ATmega328P-PU

Commit message: updated schematic
Parts:
- J1: value Conn_02x05_Counter_Clockwise -> Prog
Changed lines of the file:
@@
 P 3700 2200
 F 0 "J1" H 3750 2617 50  0000 C CNN
-F 1 "Conn_02x05_Counter_Clockwise" H 3750 2526 50  0000 C CNN
+F 1 "Prog" H 3750 2526 50  0000 C CNN
 F 2 "Connector_PinHeader_2.54mm:PinHeader_2x05_P2.54mm_Vertical" H 3700 2200 50  0001 C CNN
 F 3 "~" H 3700 2200 50  0001 C CNN
